Commit message: Update chapter 6 codes

File: chapter_6/mobile_robot_description/urdf/robot_model.xacro (robot description, xacro)
@@ -4,7 +4,7 @@
  -->
 <robot name="mobile_robot" xmlns:xacro="http://ros.org/wiki/xacro">
-  <property name="M_PI" value="3.1415926535897931" />
-  <property name="M_PI_2" value="1.570796327" />
-  <property name="DEG_TO_RAD" value="0.017453293" />
+  <xacro:property name="M_PI" value="3.1415926535897931" />
+  <xacro:property name="M_PI_2" value="1.570796327" />
+  <xacro:property name="DEG_TO_RAD" value="0.017453293" />
  <!-- <xacro:macro name="mobile_robot">   -->
     <link name="base_footprint"/>
